File: Connector_kIckad.kicad_sch (KiCad schematic)
At the start: 4 parts, among them J1 Conn_01x04_Pin, J2 Conn_01x04_Pin, J3 Conn_01x09_Pin, J4 Conn_02x03_Odd_Even

Commit message: Connector adding
Connections:
- net GND: now reaches J1.1 (Pin_1)
- net GND: now also J2.1 (Pin_1), J3.8 (Pin_8), J4.2 (Pin_2), J4.6 (Pin_6)
- net VCC: now reaches J1.2 (Pin_2)
- net VCC: now also J2.2 (Pin_2), J3.9 (Pin_9)
- net RX: now reaches J1.3 (Pin_3)
- net TX: now reaches J1.4 (Pin_4)
- net SDA: now reaches J2.3 (Pin_3)
- net SCK: now reaches J2.4 (Pin_4)
- net SCK: now also J4.3 (Pin_3)
- net D2: now reaches J3.1 (Pin_1)
- net D3: now reaches J3.2 (Pin_2)
- net D4: now reaches J3.3 (Pin_3)
- net D5: now reaches J3.4 (Pin_4)
- net D6: now reaches J3.5 (Pin_5)
- net D7: now reaches J3.6 (Pin_6)
- net D8: now reaches J3.7 (Pin_7)
- net MISO: now reaches J4.1 (Pin_1)
- net MOSI: now reaches J4.4 (Pin_4)
- net RESET: now reaches J4.5 (Pin_5)
Other:
- note added: "GPIO"
- note added: "I2C"
- note added: "ICSP"
- note added: "SERIAL UART"
- moved on the sheet: J1, J2, J3

Commit message: Changes both sheet
Parts:
- renumbered J2 to J1, J1 to J2
Changed lines of the file:
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@@
 		(dnp no)
 		(fields_autoplaced yes)
-		(property "Reference" "J1"
+		(property "Reference" "J2"
 			(at 99.695 36.83 0)
 			(effects
@@
 			(project "MCU Datalogger"
 				(path "/8c17128f-7127-4964-b664-e83d9a8ccbe4/3feca284-0ad9-4ef4-8262-f85138b1f5ba"
-					(reference "J1")
+					(reference "J2")
 					(unit 1)
 				)
@@
 		(dnp no)
 		(fields_autoplaced yes)
-		(property "Reference" "J2"
+		(property "Reference" "J1"
 			(at 65.405 36.83 0)
 			(effects
@@
 			(project ""
 				(path "/8c17128f-7127-4964-b664-e83d9a8ccbe4/3feca284-0ad9-4ef4-8262-f85138b1f5ba"
-					(reference "J2")
+					(reference "J1")
 					(unit 1)
 				)
