File: MCU Datalogger.kicad_sch (KiCad schematic)
At the start: 26 parts, among them U1 DS1337S_, U2 ATMEGA328P-AU, U3 24LC1025, U4 24LC1025, Y1 32.768 KHz, Y2 16MHz

Commit message: added connection
Connections:
- net at C5.2: now also C4.2, Y2.1
Changed lines of the file:
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@@
 		(company "Nlogoz")
+	)
+	(junction
+		(at 163.83 67.31)
+		(diameter 0)
+		(color 0 0 0 0)
+	)
+	(wire
+		(pts
+			(xy 100.33 67.31) (xy 163.83 67.31)
+		)
+		(stroke
+			(width 0)
+			(type default)
+		)
+	)
+	(wire
+		(pts
+			(xy 163.83 67.31) (xy 177.8 67.31)
+		)
+		(stroke
+			(width 0)
+			(type default)
+		)
 	)
 	(symbol

Commit message: Connector adding
Connections:
- net at D2.1 (K): now also R4.1
- net at D2.2 (A): now also BT1.1 (+), C3.1, U2.18 (AVCC), U2.4 (VCC), U2.6 (VCC)
- net at U1.1 (X1): now also Y1.1
- net at U1.2 (X2): now also Y1.2
- net at U1.3 (~{INTA}): now also R2.2
- net GND: now reaches U1.4 (GND)
- net GND: now also BT1.2 (-), C1.1, C3.2, C4.2, C5.2, C6.2, R1.1, R4.2, U2.21 (GND), U2.3 (GND), U2.5 (GND), U3.4 (GND), U3.7 (WP), U4.2 (A1), U4.4 (GND), U4.7 (WP)
- net SDA: now reaches U1.5 (SDA)
- net SDA: now also R7.2, U2.27 (PC4), U3.5 (SDA), U4.5 (SDA)
- net SCK: now reaches U1.6 (SCL)
- net SCK: now also D1.2 (A), R6.2, U2.17 (PB5), U3.6 (SCL), U4.6 (SCL)
- net at U1.7 (SQW/~INT): now also R3.2
- net VCC: now reaches U1.8 (VCC)
- net VCC: now also C4.1, R2.1, R3.1, R5.1, R6.1, R7.1, U3.1 (A0), U3.2 (A1), U3.3 (A2), U3.8 (VCC), U4.1 (A0), U4.3 (A2), U4.8 (VCC)
- net at C5.1: now also U2.7 (PB6), Y2.1
- net RESET: now reaches R5.2
- net RESET: now also U2.29 (PC6/~{RESET})
- net at C1.2: now also U2.20 (AREF)
- net at C6.1: now also U2.8 (PB7), Y2.2
- net at D1.1 (K): now also R1.2
- net D3: now reaches U2.1 (PD3)
- net D6: now reaches U2.10 (PD6)
- net D7: now reaches U2.11 (PD7)
- net D8: now reaches U2.12 (PB0)
- net MOSI: now reaches U2.15 (PB3)
- net MISO: now reaches U2.16 (PB4)
- net D4: now reaches U2.2 (PD4)
- net SCL: now reaches U2.28 (PC5)
- net RX: now reaches U2.30 (PD0)
- net TX: now reaches U2.31 (PD1)
- net D2: now reaches U2.32 (PD2)
- net D5: now reaches U2.9 (PD5)
- no-connect marks 0 -> 8
Other:
- sheet ConnectorSheet ports: added D2, D3, D4, D5, D6, D7, D8, GND, MISO, MOSI, RESET, RX, SCK, SDA, TX, VCC; removed none
- moved on the sheet: BT1, C1, C2, C3, C4, C5, C6, D1, D2, R1, R2, R3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

Commit message: Changes both sheet
Parts:
- removed C2: C_Polarized, Capacitor_SMD:C_0805_2012Metric, symbol Device:C_Polarized
- renumbered C4 to C1, C1 to C2, C5 to C4, C6 to C5, R2 to R1, R3 to R2, R1 to R3
Connections:
- net D5 is gone; now on net D3: U2.9 (PD5)
- net SCL is gone; now on net SCK: U2.28 (PC5)

Commit message: After comment
Connections:
- net D4 is gone; now on net D3: U2.2 (PD4)
Other:
- note added: "EEPROM"
- note added: "MCU"
- note added: "MOUNTING HOLE"
- note added: "REAL TIME CLOCK"
- moved on the sheet: BT1, C2, C3, C4, C5, D1, D2, H1, H2, H3, H4, R3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

Commit message: Initail Layout
Connections:
- net D3: no longer U2.2 (PD4), U2.9 (PD5)
- new net D4: U2.2 (PD4)
- new net D5: U2.9 (PD5)
Changed lines of the file:
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@@
-	)
-	(junction
-		(at 68.58 111.76)
-		(diameter 0)
-		(color 0 0 0 0)
 	)
 	(junction
@@
 	)
 	(junction
-		(at 68.58 109.22)
-		(diameter 0)
-		(color 0 0 0 0)
-	)
-	(junction
 		(at 220.98 90.17)
 		(diameter 0)
@@
 	)
 	(junction
-		(at 68.58 114.3)
-		(diameter 0)
-		(color 0 0 0 0)
-	)
-	(junction
 		(at 134.62 50.8)
 		(diameter 0)
@@
 	(wire
 		(pts
-			(xy 68.58 109.22) (xy 72.39 109.22)
-		)
-		(stroke
-			(width 0)
-			(type default)
-		)
-	)
-	(wire
-		(pts
 			(xy 76.2 39.37) (xy 78.74 39.37)
 		)
@@
 	(wire
 		(pts
-			(xy 68.58 114.3) (xy 72.39 114.3)
-		)
-		(stroke
-			(width 0)
-			(type default)
-		)
-	)
-	(wire
-		(pts
 			(xy 76.2 46.99) (xy 76.2 52.07)
 		)
@@
 	(wire
 		(pts
-			(xy 77.47 58.42) (xy 77.47 64.77)
+			(xy 77.47 62.23) (xy 77.47 64.77)
 		)
 		(stroke
@@
 	(wire
 		(pts
-			(xy 76.2 58.42) (xy 77.47 58.42)
+			(xy 76.2 62.23) (xy 77.47 62.23)
 		)
 		(stroke
@@
 	(wire
 		(pts
-			(xy 68.58 111.76) (xy 72.39 111.76)
-		)
-		(stroke
-			(width 0)
-			(type default)
-		)
-	)
-	(wire
-		(pts
 			(xy 43.18 97.79) (xy 46.99 97.79)
 		)
@@
 	(wire
 		(pts
-			(xy 68.58 109.22) (xy 68.58 111.76)
-		)
-		(stroke
-			(width 0)
-			(type default)
-		)
-	)
-	(wire
-		(pts
-			(xy 68.58 111.76) (xy 68.58 114.3)
-		)
-		(stroke
-			(width 0)
-			(type default)
-		)
-	)
-	(wire
-		(pts
 			(xy 223.52 44.45) (xy 223.52 46.99)
-		)
-		(stroke
-			(width 0)
-			(type default)
-		)
-	)
-	(wire
-		(pts
-			(xy 76.2 58.42) (xy 76.2 62.23)
 		)
 		(stroke
@@
 	)
 	(label "D3"
-		(at 71.12 109.22 0)
+		(at 68.58 109.22 0)
 		(fields_autoplaced yes)
 		(effects
@@
 	)
 	(label "D4"
-		(at 71.12 111.76 0)
+		(at 68.58 111.76 0)
 		(fields_autoplaced yes)
 		(effects
@@
 	)
 	(label "D5"
-		(at 71.12 114.3 0)
-		(fields_autoplaced yes)
-		(effects
+		(at 68.58 114.3 0)
+		(fields_autoplaced yes)
+		(effects

Commit message: Layout complete
Connections:
- net VCC: now also BT1.1 (+), C3.1, D2.2 (A), U2.18 (AVCC), U2.4 (VCC), U2.6 (VCC)
Changed lines of the file:
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@@
+		)
+	)
+	(label "VCC"
+		(at 240.03 41.91 0)
+		(fields_autoplaced yes)
+		(effects
+			(font
+				(size 1.27 1.27)
+			)
+			(justify left bottom)
 		)
 	)
