File: _autosave-MCU Datalogger.kicad_pcb (KiCad board)
At the start: 2 copper layers, 50 x 30 mm, 31 parts, among them J1 Conn_01x04_Pin, J2 Conn_01x04_Pin, J3 Conn_01x09_Pin, J4 Conn_02x03_Odd_Even, U1 DS1337S_, U2 ATMEGA328P-AU, U3 24LC1025, U4 24LC1025, Y1 32.768 KHz, Y2 16MHz

Commit message: GARBER FILE
Other:
- board text added: "0.0000 mm / 0.0000 mm"
- board text added: "0.3000 mm"
- board text added: "1.6000 mm"
- board text added: "50.0044 mm x 30.0027 mm"
- board text added: "BOARD CHARACTERISTICS"
- board text added: "Board Thickness:"
- board text added: "Board overall dimensions:"
- board text added: "Castellated pads:"
- board text added: "Copper Finish:"
- board text added: "Copper Layer Count:"
- board text added: "Edge card connectors:"
- board text added: "Impedance Control:"
- board text added: "Min hole diameter:"
- board text added: "Min track/spacing:"
- board text added: "No"
- board text added: "None"
- board text added: "Plated Board Edge:"
